Commit message: gazebo sim working

File: description/robot.urdf.xacro (robot description, xacro)
@@ -2,3 +2,4 @@
 <robot xmlns:xacro="http://www.ros.org/wiki/xacro"  name="robot">
     <xacro:include filename="robot_core.xacro" />
+    <xacro:include filename="gazebo_control.xacro" />
 </robot>

File: description/robot_core.xacro (robot description, xacro)
@@ -2,5 +2,5 @@
 <robot xmlns:xacro="http://www.ros.org/wiki/xacro" >
     <xacro:include filename="inertial_macros.xacro"/>
-    <xacro:property name="chassis_length" value="-0.140"/>
+    <xacro:property name="chassis_length" value="0.140"/>
     <xacro:property name="chassis_width" value="0.165"/>  <!-- good-->
     <xacro:property name="chassis_height" value="0.138"/>
@@ -9,10 +9,10 @@
     <xacro:property name="wheel_thickness" value="0.026"/>
     <xacro:property name="wheel_mass" value="0.05"/>
-    <xacro:property name="wheel_offset_x" value="-0.100"/>
+    <xacro:property name="wheel_offset_x" value="0.100"/>
     <xacro:property name="wheel_offset_y" value="-0.1010"/>
     <xacro:property name="wheel_offset_z" value="-0.01"/>
     <xacro:property name="caster_wheel_radius" value="0.033"/>
     <xacro:property name="caster_wheel_mass" value="0.01"/>
-    <xacro:property name="caster_wheel_offset_x" value="-0.030"/>
+    <xacro:property name="caster_wheel_offset_x" value="0.030"/>
     <xacro:property name="caster_wheel_offset_z" value="${wheel_offset_z - wheel_radius + caster_wheel_radius}"/>
     <material name="white">
