Commit message: urdf update

File: description/lidar.xacro (robot description, xacro)
@@ -4,5 +4,5 @@
         <parent link="chassis"/>
         <child link="laser_frame"/>
-        <origin xyz="0.10 0 0.150" rpy="0 0 0"/>
+        <origin xyz="0.20 0 0.150" rpy="0 0 0"/>
     </joint>
     <link name="laser_frame">

File: description/robot_core.xacro (robot description, xacro)
@@ -2,17 +2,17 @@
 <robot xmlns:xacro="http://www.ros.org/wiki/xacro" >
     <xacro:include filename="inertial_macros.xacro"/>
-    <xacro:property name="chassis_length" value="0.140"/>
-    <xacro:property name="chassis_width" value="0.165"/>  <!-- good-->
+    <xacro:property name="chassis_length" value="0.250"/>
+    <xacro:property name="chassis_width" value="0.300"/>  <!-- good-->
     <xacro:property name="chassis_height" value="0.138"/>
     <xacro:property name="chassis_mass" value="1.0"/>
-    <xacro:property name="wheel_radius" value="0.033"/>
+    <xacro:property name="wheel_radius" value="0.035"/>
     <xacro:property name="wheel_thickness" value="0.026"/>
     <xacro:property name="wheel_mass" value="0.05"/>
-    <xacro:property name="wheel_offset_x" value="0.100"/>
-    <xacro:property name="wheel_offset_y" value="-0.1010"/>
+    <xacro:property name="wheel_offset_x" value="0.05"/>
+    <xacro:property name="wheel_offset_y" value="-0.1650"/>
     <xacro:property name="wheel_offset_z" value="-0.01"/>
-    <xacro:property name="caster_wheel_radius" value="0.033"/>
+    <xacro:property name="caster_wheel_radius" value="0.035"/>
     <xacro:property name="caster_wheel_mass" value="0.01"/>
-    <xacro:property name="caster_wheel_offset_x" value="0.030"/>
+    <xacro:property name="caster_wheel_offset_x" value="0.20"/>
     <xacro:property name="caster_wheel_offset_z" value="${wheel_offset_z - wheel_radius + caster_wheel_radius}"/>
     <material name="white">
@@ -54,5 +54,5 @@
                 <box size="${chassis_length} ${chassis_width} ${chassis_height}"/>
             </geometry>
-            <material name="orange"/>
+            <material name="blue"/>
         </visual>
         <collision>
@@ -67,5 +67,5 @@
     </link>
     <gazebo reference="chassis">
-        <material>Gazebo/Orange</material>
+        <material>Gazebo/Blue</material>
     </gazebo>
     <!-- LEFT WHEEL LINK -->
@@ -81,5 +81,5 @@
                 <cylinder radius="${wheel_radius}" length="${wheel_thickness}"/>
             </geometry>
-            <material name="blue"/>
+            <material name="black"/>
         </visual>
         <collision>
@@ -93,5 +93,5 @@
     </link>
     <gazebo reference="left_wheel">
-        <material>Gazebo/Blue</material>
+        <material>Gazebo/Black</material>
     </gazebo>
     <!-- RIGHT WHEEL LINK -->
@@ -107,5 +107,5 @@
                 <cylinder radius="${wheel_radius}" length="${wheel_thickness}"/>
             </geometry>
-            <material name="blue"/>
+            <material name="black"/>
         </visual>
         <collision>
@@ -119,5 +119,5 @@
     </link>
     <gazebo reference="right_wheel">
-        <material>Gazebo/Blue</material>
+        <material>Gazebo/Black</material>
     </gazebo>
     <!-- CASTER WHEEL LINK -->

Commit message: Update lidar.xacro

File: description/lidar.xacro (robot description, xacro)
@@ -3,8 +3,8 @@
     <joint name="laser_joint" type="fixed">
         <parent link="chassis"/>
-        <child link="laser_frame"/>
+        <child link="laser"/>
         <origin xyz="0.20 0 0.150" rpy="0 0 0"/>
     </joint>
-    <link name="laser_frame">
+    <link name="laser">
         <visual>
             <geometry>
@@ -29,5 +29,5 @@
         </xacro:inertial_cylinder>
     </link>
-    <gazebo reference="laser_frame">
+    <gazebo reference="laser">
         <material>Gazebo/Black</material>
         <sensor name="laser" type="ray">
@@ -53,5 +53,5 @@
                 </ros>
                 <output_type>sensor_msgs/LaserScan</output_type>
-                <frame_name>laser_frame</frame_name>
+                <frame_name>laser</frame_name>
             </plugin>
         </sensor>
